File: synth-vco/synth-vco.kicad_pcb (KiCad board)
At the start: 4 copper layers, 91.8 x 61.8 mm, 148 parts, among them J1 Conn_Coaxial, J2 Screw_Terminal_01x02, J3 61202021621, J4 Conn_Coaxial, U1 ADF4158, U10 LT3045IMSE_TRPBF, U11 LT3045IMSE_TRPBF, U12 LT3045IMSE_TRPBF, U13 LT8570EMS8E_TRPBF, U14 LT3065EDDPBF, U15 LT3065EDDPBF, U16 BT09E, U3 ADP-2-10+, U4 DAT-15R5A-SP+, U5 OPA192IDGKT, U6 TPSM53602RDAR, U7 LT3045IMSE_TRPBF, U8 LT3045IMSE_TRPBF, U9 LT3045IMSE_TRPBF, Y1 FT3MN 26 MHz, Y3 CVCO55CW-0500-1000

Commit message: feat: silkscreen edits + art
Parts:
- added G***: LOGO, LOGO, F.Cu at (157.1, 61.2)
- added G***: LOGO, LOGO, F.Cu at (176.4, 110.7)
- added G***: LOGO, LOGO, F.Cu at (137.9, 62.4)
Other:
- board text added: "+12V"
- board text added: "A_CLK"
- board text added: "A_DAT"
- board text added: "A_LE"
- board text added: "FMCW CHIRP SOURCE"
- board text added: "GND"
- board text added: "PLL synth + TX/LO amps Rev A"
- board text added: "P_CE"
- board text added: "P_CLK"
- board text added: "P_DAT"
- board text added: "P_LE"
- board text added: "P_MUX"
- board text added: "P_TXDAT"

Commit message: feat: silkscreen
Parts:
- removed the G*** at (137.9, 62.4)
Changed lines of the file:
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@@
 		(embedded_fonts no)
 	)
-	(footprint "LOGO"
-		(layer "F.Cu")
-		(at 137.9 62.4 -10)
-		(property "Reference" "G***"
-			(at 0 0 170)
-			(layer "F.SilkS")
-			(hide yes)
-			(effects
-				(font
-					(size 1.5 1.5)
-					(thickness 0.3)
-				)
-			)
-		)
-		(property "Value" "LOGO"
-			(at 0.749999 0 170)
-			(layer "F.SilkS")
-			(hide yes)
-			(effects
-				(font
-					(size 1.5 1.5)
-					(thickness 0.3)
-				)
-			)
-		)
-		(property "Datasheet" ""
-			(at 0 0 170)
-			(layer "F.Fab")
-			(hide yes)
-			(effects
-				(font
-					(size 1.27 1.27)
-				)
-			)
-		)
-		(property "Description" ""
-			(at 0 0 170)
-			(layer "F.Fab")
-			(hide yes)
-			(effects
-				(font
-					(size 1.27 1.27)
-				)
-			)
-		)
-		(attr board_only exclude_from_pos_files exclude_from_bom)
-		(duplicate_pad_numbers_are_jumpers no)
-		(fp_poly
-			(pts
-				(xy -5.024615 1.181782) (xy -5.050546 1.199611) (xy -5.075634 1.208559) (xy -5.104078 1.210889)
-				(xy -5.106848 1.203286) (xy -5.080917 1.185459) (xy -5.055827 1.176512) (xy -5.027385 1.17418)
-			)
-			(stroke
-				(width 0)
-				(type solid)
-			)
-			(fill yes)
-			(layer "F.SilkS")
-		)
-		(fp_poly
-			(pts
-				(xy 5.157463 -2.348314) (xy 5.140279 -2.332762) (xy 5.098207 -2.313666) (xy 5.091211 -2.311188)
-				(xy 4.867277 -2.233729) (xy 4.679318 -2.167184) (xy 4.528262 -2.111883) (xy 4.415023 -2.068159)
-				(xy 4.393017 -2.059194) (xy 4.312709 -2.02684) (xy 4.202085 -1.983431) (xy 4.069093 -1.93201) (xy 3.921677 -1.875609)
-				(xy 3.767781 -1.817271) (xy 3.615348 -1.760029) (xy 3.472325 -1.706924) (xy 3.455295 -1.700651)
-				(xy 3.360735 -1.665664) (xy 3.267307 -1.63078) (xy 3.190707 -1.601866) (xy 3.169903 -1.593909) (xy 3.124133 -1.576296)
-				(xy 3.046374 -1.546378) (xy 2.942679 -1.506485) (xy 2.819109 -1.458947) (xy 2.681727 -1.406097)
-				(xy 2.536587 -1.350265) (xy 2.527768 -1.346872) (xy 2.381636 -1.290497) (xy 2.242293 -1.236437)
-				(xy 2.11594 -1.187122) (xy 2.00878 -1.144983) (xy 1.927014 -1.112448) (xy 1.876847 -1.091947) (xy 1.875439 -1.09135)
-				(xy 1.817363 -1.067126) (xy 1.730964 -1.031714) (xy 1.6258 -0.989002) (xy 1.511429 -0.942879) (xy 1.448966 -0.917832)
-				(xy 1.325875 -0.868325) (xy 1.18938 -0.813013) (xy 1.046604 -0.754823) (xy 0.904671 -0.696682) (xy 0.770708 -0.641517)
-				(xy 0.65184 -0.592258) (xy 0.555191 -0.55183) (xy 0.487886 -0.52316) (xy 0.479051 -0.519305) (xy 0.242226 -0.414221)
-				(xy 0.003063 -0.306045) (xy -0.234298 -0.196779) (xy -0.465729 -0.088417) (xy -0.687101 0.017043)
-				(xy -0.894279 0.1176) (xy -1.083131 0.211258) (xy -1.24953 0.296021) (xy -1.38934 0.369888) (xy -1.49843 0.430862)
-				(xy -1.549279 0.461599) (xy -1.787845 0.627026) (xy -2.002643 0.805092) (xy -2.187577 0.990373)
-				(xy -2.306865 1.135997) (xy -2.38038 1.250135) (xy -2.455467 1.392932) (xy -2.526836 1.552856) (xy -2.5892 1.718372)
-				(xy -2.622683 1.824477) (xy -2.651236 1.929311) (xy -2.680622 2.047139) (xy -2.708899 2.168999)
-				(xy -2.734122 2.285934) (xy -2.754343 2.388978) (xy -2.767617 2.469167) (xy -2.771984 2.512479)
-				(xy -2.787277 2.527684) (xy -2.787681 2.527689) (xy -2.793476 2.508475) (xy -2.799051 2.455701)
-				(xy -2.803895 2.376578) (xy -2.807496 2.278314) (xy -2.808473 2.235291) (xy -2.811809 2.116736)
-				(xy -2.817027 2.000216) (xy -2.82346 1.897926) (xy -2.830435 1.822065) (xy -2.831667 1.812378) (xy -2.869563 1.612996)
-				(xy -2.925692 1.430661) (xy -2.997558 1.270218) (xy -3.082665 1.136511) (xy -3.178522 1.034386)
-				(xy -3.260894 0.97887) (xy -3.371 0.938361) (xy -3.51023 0.911489) (xy -3.669067 0.898846) (xy -3.838007 0.901032)
-				(xy -4.007542 0.918642) (xy -4.064821 0.928474) (xy -4.323012 0.982496) (xy -4.569144 1.043139)
-				(xy -4.779024 1.103787) (xy -4.85876 1.127918) (xy -4.922498 1.145334) (xy -4.961309 1.153692) (xy -4.968775 1.153591)
-				(xy -4.954823 1.142013) (xy -4.91121 1.116198) (xy -4.8448 1.080023) (xy -4.766237 1.039275) (xy -4.681105 0.995638)
-				(xy -4.608772 0.957809) (xy -4.557379 0.930093) (xy -4.535715 0.917331) (xy -4.508675 0.900648)
-				(xy -4.456453 0.870899) (xy -4.389827 0.834213) (xy -4.382825 0.830419) (xy -4.155575 0.70553) (xy -3.95782 0.592218)
-				(xy -3.78178 0.485562) (xy -3.619673 0.380633) (xy -3.463714 0.272503) (xy -3.306124 0.156247) (xy -3.248851 0.1125)
-				(xy -3.11144 -0.00791) (xy -2.985371 -0.150204) (xy -2.868069 -0.318383) (xy -2.756955 -0.516451)
-				(xy -2.649456 -0.748411) (xy -2.573208 -0.937721) (xy -2.485795 -1.179332) (xy -2.405289 -1.430587)
-				(xy -2.33212 -1.686879) (xy -2.314195 -1.710609) (xy -2.307171 -1.71236) (xy -2.299264 -1.693311)
-				(xy -2.291125 -1.641464) (xy -2.283714 -1.564779) (xy -2.278074 -1.472833) (xy -2.260975 -1.272423)
-				(xy -2.228461 -1.104512) (xy -2.178384 -0.96306) (xy -2.108592 -0.842013) (xy -2.01694 -0.735323)
-				(xy -2.015583 -0.733994) (xy -1.93785 -0.664593) (xy -1.867282 -0.619176) (xy -1.788303 -0.587889)
-				(xy -1.781153 -0.585701) (xy -1.651979 -0.558211) (xy -1.524035 -0.551227) (xy -1.412703 -0.565397)
-				(xy -1.397838 -0.569557) (xy -1.358533 -0.580449) (xy -1.287126 -0.599143) (xy -1.191107 -0.623725)
-				(xy -1.077968 -0.652273) (xy -0.958106 -0.682153) (xy -0.790047 -0.723809) (xy -0.65588 -0.757126)
-				(xy -0.549923 -0.783557) (xy -0.466494 -0.804549) (xy -0.399905 -0.821554) (xy -0.344472 -0.83602)
-				(xy -0.294514 -0.849398) (xy -0.244347 -0.863141) (xy -0.19366 -0.877201) (xy -0.098951 -0.902925)
-				(xy -0.002398 -0.928141) (xy 0.076309 -0.947722) (xy 0.08154 -0.948959) (xy 0.170835 -0.971438)
-				(xy 0.267422 -0.997866) (xy 0.305778 -1.009071) (xy 0.395637 -1.0344) (xy 0.493321 -1.059493) (xy 0.531878 -1.068594)
-				(xy 0.597993 -1.084949) (xy 0.648528 -1.09997) (xy 0.6673 -1.107651) (xy 0.697281 -1.118715) (xy 0.754253 -1.13446)
-				(xy 0.818327 -1.149741) (xy 0.910107 -1.171578) (xy 1.006718 -1.196705) (xy 1.060031 -1.211733)
-				(xy 1.30926 -1.282607) (xy 1.508507 -1.335505) (xy 1.634828 -1.368767) (xy 1.798977 -1.413497) (xy 1.999753 -1.469372)
-				(xy 2.02833 -1.477394) (xy 2.115721 -1.501724) (xy 2.206323 -1.526606) (xy 2.252566 -1.539133) (xy 2.325041 -1.55884)
-				(xy 2.416805 -1.584127) (xy 2.507383 -1.609346) (xy 2.644154 -1.647611) (xy 2.749461 -1.676902)
-				(xy 2.831068 -1.699338) (xy 2.896742 -1.717044) (xy 2.95425 -1.732138) (xy 2.996627 -1.743008) (xy 3.083594 -1.765844)
-				(xy 3.174815 -1.790854) (xy 3.210672 -1.801055) (xy 3.300364 -1.826609) (xy 3.415088 -1.858681)
-				(xy 3.540478 -1.893304) (xy 3.662171 -1.926501) (xy 3.740688 -1.947624) (xy 3.822821 -1.970311)
-				(xy 3.914801 -1.996817) (xy 3.954734 -2.008706) (xy 4.044057 -2.034521) (xy 4.140669 -2.060731)
-				(xy 4.178972 -2.070548) (xy 4.331235 -2.109172) (xy 4.446093 -2.139828) (xy 4.525978 -2.1632) (xy 4.573325 -2.179961)
-				(xy 4.576484 -2.181355) (xy 4.613685 -2.194987) (xy 4.678841 -2.215847) (xy 4.760593 -2.240356)
-				(xy 4.80072 -2.251896) (xy 4.893831 -2.278831) (xy 4.98295 -2.305525) (xy 5.053118 -2.32747) (xy 5.070826 -2.333327)
-				(xy 5.122323 -2.347965) (xy 5.153355 -2.351299)
-			)
-			(stroke
-				(width 0)
-				(type solid)
-			)
-			(fill yes)
-			(layer "F.SilkS")
-		)
-		(embedded_fonts no)
-	)
 	(footprint "Capacitor_SMD:C_0603_1608Metric_Pad1.08x0.95mm_HandSolder"
 		(layer "F.Cu")
@@
 		(stroke
 			(width 0.05)
-			(type solid)
+			(type dash_dot_dot)
 		)
 		(fill no)
